File: Prototype/PCB/Pingboard_Prototype.sch (KiCad schematic (older format))
At the start: 22 parts, among them J1 Conn_01x02, J2 Conn_01x04, J3 Conn_01x02, SW1 SW_Push, SW2 SW_Push, SW3 SW_Push, SW4 SW_Push, U1 TLC59108xPW, U2 TLC59108xPW

Commit message: Draft 2
Parts:
- added D5: gn, LED_SMD:LED_0603_1608Metric_Pad1.05x0.95mm_HandSolder, symbol Device:LED
- added R7: 580, Resistor_SMD:R_0603_1608Metric_Pad0.98x0.95mm_HandSolder, symbol Device:R
- C3: footprint Capacitor_SMD:C_0201_0603Metric_Pad0.64x0.40mm_HandSolder -> Capacitor_SMD:C_0603_1608Metric_Pad1.08x0.95mm_HandSolder
- D1: Digikey (none) -> https://www.digikey.de/product-detail/de/broadcom-limited/A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
- D2: Digikey (none) -> https://www.digikey.de/product-detail/de/broadcom-limited/A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; Farnell (none) -> https://de.farnell.com/broadcom-limited/asmb-ktf0-0a306/led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
- D3, D4: Farnell (none) -> https://de.farnell.com/broadcom-limited/asmb-ktf0-0a306/led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
- R5, R6: value 720 -> Rext
- U1: Digikey (none) -> https://www.digikey.de/product-detail/de/texas-instruments/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
Connections:
- wire segments 135 -> 149
- no-connect marks 0 -> 4
Other:
- moved on the sheet: C1, C2, C3, D1, D2, D3, D4, R1, R2, R3, R4, R5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

Commit message: Draft 3
Parts:
- J1, J3: footprint Connector_PinHeader_2.54mm:PinHeader_1x02_P2.54mm_Vertical -> Connector_PinHeader_1.27mm:PinHeader_1x02_P1.27mm_Vertical
- J2: footprint Connector_PinHeader_2.54mm:PinHeader_1x04_P2.54mm_Vertical -> Connector_PinHeader_1.27mm:PinHeader_1x04_P1.27mm_Vertical
Other:
- moved on the sheet: R7
Changed lines of the file:
@@
 F 0 "J2" H 3918 2175 50  0000 C CNN
 F 1 "Conn_01x04" H 3918 2266 50  0000 C CNN
-F 2 "Connector_PinHeader_2.54mm:PinHeader_1x04_P2.54mm_Vertical" H 4000 2600 50  0001 C CNN
+F 2 "Connector_PinHeader_1.27mm:PinHeader_1x04_P1.27mm_Vertical" H 4000 2600 50  0001 C CNN
 F 3 "~" H 4000 2600 50  0001 C CNN
 	1    4000 2600
@@
 F 0 "J1" H 2018 1675 50  0000 C CNN
 F 1 "Conn_01x02" H 2018 1766 50  0000 C CNN
-F 2 "Connector_PinHeader_2.54mm:PinHeader_1x02_P2.54mm_Vertical" H 2100 2000 50  0001 C CNN
+F 2 "Connector_PinHeader_1.27mm:PinHeader_1x02_P1.27mm_Vertical" H 2100 2000 50  0001 C CNN
 F 3 "~" H 2100 2000 50  0001 C CNN
 	1    2100 2000
@@
 F 0 "J3" H 3968 1525 50  0000 C CNN
 F 1 "Conn_01x02" H 3968 1616 50  0000 C CNN
-F 2 "Connector_PinHeader_2.54mm:PinHeader_1x02_P2.54mm_Vertical" H 4050 1850 50  0001 C CNN
+F 2 "Connector_PinHeader_1.27mm:PinHeader_1x02_P1.27mm_Vertical" H 4050 1850 50  0001 C CNN
 F 3 "~" H 4050 1850 50  0001 C CNN
 	1    4050 1850
@@
 L Device:R R7
 U 1 1 5FAF1606
-P 3200 2200
-F 0 "R7" H 3130 2154 50  0000 R CNN
-F 1 "580" H 3130 2245 50  0000 R CNN
-F 2 "Resistor_SMD:R_0603_1608Metric_Pad0.98x0.95mm_HandSolder" V 3130 2200 50  0001 C CNN
-F 3 "~" H 3200 2200 50  0001 C CNN
-	1    3200 2200
-	-1   0    0    1
-$EndComp
-$Comp
-L Device:LED D5
-U 1 1 5FAF1F7A
 P 3200 1850
-F 0 "D5" V 3147 1930 50  0000 L CNN
-F 1 "gn" V 3238 1930 50  0000 L CNN
-F 2 "LED_SMD:LED_0603_1608Metric_Pad1.05x0.95mm_HandSolder" H 3200 1850 50  0001 C CNN
+F 0 "R7" H 3130 1804 50  0000 R CNN
+F 1 "580" H 3130 1895 50  0000 R CNN
+F 2 "Resistor_SMD:R_0603_1608Metric_Pad0.98x0.95mm_HandSolder" V 3130 1850 50  0001 C CNN
 F 3 "~" H 3200 1850 50  0001 C CNN
 	1    3200 1850
-	0    1    1    0
+	-1   0    0    1
 $EndComp
 Wire Wire Line
 	3200 2350 3200 2400
-Wire Wire Line
-	3200 2000 3200 2050
 Wire Wire Line
 	3200 1650 3200 1700
@@
 	8600 2500 8600 2550
 Connection ~ 8600 2550
+$Comp
+L Device:LED D5
+U 1 1 5FAF1F7A
+P 3200 2200
+F 0 "D5" V 3147 2280 50  0000 L CNN
+F 1 "gn" V 3238 2280 50  0000 L CNN
+F 2 "LED_SMD:LED_0603_1608Metric_Pad1.05x0.95mm_HandSolder" H 3200 2200 50  0001 C CNN
+F 3 "~" H 3200 2200 50  0001 C CNN
+	1    3200 2200
+	0    -1   -1   0
+$EndComp
+Wire Wire Line
+	3200 2000 3200 2050
 $EndSCHEMATC

Commit message: Draft 4
Arduino Huckepack
Parts:
- removed D5: gn, LED_SMD:LED_0603_1608Metric_Pad1.05x0.95mm_HandSolder, symbol Device:LED
- removed J1, J3: Conn_01x02, Connector_PinHeader_1.27mm:PinHeader_1x02_P1.27mm_Vertical, symbol Connector_Generic:Conn_01x02
- removed J2: Conn_01x04, Connector_PinHeader_1.27mm:PinHeader_1x04_P1.27mm_Vertical, symbol Connector_Generic:Conn_01x04
- removed R7: 580, Resistor_SMD:R_0603_1608Metric_Pad0.98x0.95mm_HandSolder, symbol Device:R
- added J1, J2: Conn_01x12, Connector_PinHeader_2.54mm:PinHeader_1x12_P2.54mm_Vertical, symbol Connector_Generic:Conn_01x12
Connections:
- wire segments 149 -> 144
- no-connect marks 4 -> 17
Other:
- moved on the sheet: C3, R1, R2, R3, R4, SW1, SW2, SW3, SW4

Commit message: Draft 5
Parts:
- added U3: 74LVC1G10, Package_TO_SOT_SMD:SOT-363_SC-70-6_Handsoldering, symbol 74xGxx:74LVC1G10
Connections:
- net GND: now also U3.2 (GND)
- net Switch1: now also U3.1
- net Switch2: now also U3.3
- net Switch3: now also U3.6
- net VCC: now also U3.5 (VCC)
- net RST: now reaches J2.3 (Pin_3)
- net RST: now also U3.4
Other:
- moved on the sheet: R1, R2, R3, R4, SW1, SW2, SW3, SW4
Changed lines of the file:
@@
 L power:GND #PWR0101
 U 1 1 5FADA0BB
-P 3700 6300
-F 0 "#PWR0101" H 3700 6050 50  0001 C CNN
-F 1 "GND" H 3705 6127 50  0000 C CNN
-F 2 "" H 3700 6300 50  0001 C CNN
-F 3 "" H 3700 6300 50  0001 C CNN
-	1    3700 6300
-	1    0    0    -1
-$EndComp
-Text GLabel 2400 4800 0    39   Output ~ 0
+P 2600 6850
+F 0 "#PWR0101" H 2600 6600 50  0001 C CNN
+F 1 "GND" H 2605 6677 50  0000 C CNN
+F 2 "" H 2600 6850 50  0001 C CNN
+F 3 "" H 2600 6850 50  0001 C CNN
+	1    2600 6850
+	1    0    0    -1
+$EndComp
+Text GLabel 1300 5350 0    39   Output ~ 0
 Switch1
-Text GLabel 2400 5250 0    39   Output ~ 0
+Text GLabel 1300 5800 0    39   Output ~ 0
 Switch2
-Text GLabel 2400 5700 0    39   Output ~ 0
+Text GLabel 1300 6250 0    39   Output ~ 0
 Switch3
-Text GLabel 2400 6150 0    39   Output ~ 0
+Text GLabel 1300 6700 0    39   Output ~ 0
 Switch4
 Text GLabel 1450 2000 2    39   Input ~ 0
@@
 L Switch:SW_Push SW1
 U 1 1 5FADF5D5
-P 2950 4800
-F 0 "SW1" H 2950 5085 50  0000 C CNN
-F 1 "SW_Push" H 2950 4994 50  0000 C CNN
-F 2 "Button_Switch_Keyboard:SW_Cherry_MX_1.00u_PCB" H 2950 5000 50  0001 C CNN
-F 3 "~" H 2950 5000 50  0001 C CNN
-	1    2950 4800
+P 1850 5350
+F 0 "SW1" H 1850 5635 50  0000 C CNN
+F 1 "SW_Push" H 1850 5544 50  0000 C CNN
+F 2 "Button_Switch_Keyboard:SW_Cherry_MX_1.00u_PCB" H 1850 5550 50  0001 C CNN
+F 3 "~" H 1850 5550 50  0001 C CNN
+	1    1850 5350
 	1    0    0    -1
 $EndComp
@@
 L Switch:SW_Push SW2
 U 1 1 5FAE07D3
-P 2950 5250
-F 0 "SW2" H 2950 5535 50  0000 C CNN
-F 1 "SW_Push" H 2950 5444 50  0000 C CNN
-F 2 "Button_Switch_Keyboard:SW_Cherry_MX_1.00u_PCB" H 2950 5450 50  0001 C CNN
-F 3 "~" H 2950 5450 50  0001 C CNN
-	1    2950 5250
+P 1850 5800
+F 0 "SW2" H 1850 6085 50  0000 C CNN
+F 1 "SW_Push" H 1850 5994 50  0000 C CNN
+F 2 "Button_Switch_Keyboard:SW_Cherry_MX_1.00u_PCB" H 1850 6000 50  0001 C CNN
+F 3 "~" H 1850 6000 50  0001 C CNN
+	1    1850 5800
 	1    0    0    -1
 $EndComp
@@
 L Switch:SW_Push SW3
 U 1 1 5FAE0AC7
-P 2950 5700
-F 0 "SW3" H 2950 5985 50  0000 C CNN
-F 1 "SW_Push" H 2950 5894 50  0000 C CNN
-F 2 "Button_Switch_Keyboard:SW_Cherry_MX_1.00u_PCB" H 2950 5900 50  0001 C CNN
-F 3 "~" H 2950 5900 50  0001 C CNN
-	1    2950 5700
+P 1850 6250
+F 0 "SW3" H 1850 6535 50  0000 C CNN
+F 1 "SW_Push" H 1850 6444 50  0000 C CNN
+F 2 "Button_Switch_Keyboard:SW_Cherry_MX_1.00u_PCB" H 1850 6450 50  0001 C CNN
+F 3 "~" H 1850 6450 50  0001 C CNN
+	1    1850 6250
 	1    0    0    -1
 $EndComp
@@
 L Switch:SW_Push SW4
 U 1 1 5FAE0E9C
-P 2950 6150
-F 0 "SW4" H 2950 6435 50  0000 C CNN
-F 1 "SW_Push" H 2950 6344 50  0000 C CNN
-F 2 "Button_Switch_Keyboard:SW_Cherry_MX_1.00u_PCB" H 2950 6350 50  0001 C CNN
-F 3 "~" H 2950 6350 50  0001 C CNN
-	1    2950 6150
+P 1850 6700
+F 0 "SW4" H 1850 6985 50  0000 C CNN
+F 1 "SW_Push" H 1850 6894 50  0000 C CNN
+F 2 "Button_Switch_Keyboard:SW_Cherry_MX_1.00u_PCB" H 1850 6900 50  0001 C CNN
+F 3 "~" H 1850 6900 50  0001 C CNN
+	1    1850 6700
 	1    0    0    -1
 $EndComp
@@
 L power:VCC #PWR0104
 U 1 1 5FADAFC9
-P 3500 4450
-F 0 "#PWR0104" H 3500 4300 50  0001 C CNN
-F 1 "VCC" H 3515 4623 50  0000 C CNN
-F 2 "" H 3500 4450 50  0001 C CNN
-F 3 "" H 3500 4450 50  0001 C CNN
-	1    3500 4450
+P 2400 5000
+F 0 "#PWR0104" H 2400 4850 50  0001 C CNN
+F 1 "VCC" H 2415 5173 50  0000 C CNN
+F 2 "" H 2400 5000 50  0001 C CNN
+F 3 "" H 2400 5000 50  0001 C CNN
+	1    2400 5000
 	1    0    0    -1
 $EndComp
@@
 L Device:R R1
 U 1 1 5FADB9E3
-P 3300 4700
-F 0 "R1" V 3093 4700 50  0000 C CNN
-F 1 "4k7" V 3184 4700 50  0000 C CNN
-F 2 "Resistor_SMD:R_0603_1608Metric_Pad0.98x0.95mm_HandSolder" V 3230 4700 50  0001 C CNN
-F 3 "~" H 3300 4700 50  0001 C CNN
-	1    3300 4700
+P 2200 5250
+F 0 "R1" V 1993 5250 50  0000 C CNN
+F 1 "4k7" V 2084 5250 50  0000 C CNN
+F 2 "Resistor_SMD:R_0603_1608Metric_Pad0.98x0.95mm_HandSolder" V 2130 5250 50  0001 C CNN
+F 3 "~" H 2200 5250 50  0001 C CNN
+	1    2200 5250
 	0    1    1    0
 $EndComp
@@
 L Device:R R2
 U 1 1 5FADC3CF
-P 3300 5150
-F 0 "R2" V 3093 5150 50  0000 C CNN
-F 1 "4k7" V 3184 5150 50  0000 C CNN
-F 2 "Resistor_SMD:R_0603_1608Metric_Pad0.98x0.95mm_HandSolder" V 3230 5150 50  0001 C CNN
-F 3 "~" H 3300 5150 50  0001 C CNN
-	1    3300 5150
+P 2200 5700
+F 0 "R2" V 1993 5700 50  0000 C CNN
+F 1 "4k7" V 2084 5700 50  0000 C CNN
+F 2 "Resistor_SMD:R_0603_1608Metric_Pad0.98x0.95mm_HandSolder" V 2130 5700 50  0001 C CNN
+F 3 "~" H 2200 5700 50  0001 C CNN
+	1    2200 5700
 	0    1    1    0
 $EndComp
@@
 L Device:R R3
 U 1 1 5FADC763
-P 3300 5600
-F 0 "R3" V 3093 5600 50  0000 C CNN
-F 1 "4k7" V 3184 5600 50  0000 C CNN
-F 2 "Resistor_SMD:R_0603_1608Metric_Pad0.98x0.95mm_HandSolder" V 3230 5600 50  0001 C CNN
-F 3 "~" H 3300 5600 50  0001 C CNN
-	1    3300 5600
+P 2200 6150
+F 0 "R3" V 1993 6150 50  0000 C CNN
+F 1 "4k7" V 2084 6150 50  0000 C CNN
+F 2 "Resistor_SMD:R_0603_1608Metric_Pad0.98x0.95mm_HandSolder" V 2130 6150 50  0001 C CNN
+F 3 "~" H 2200 6150 50  0001 C CNN
+	1    2200 6150
 	0    1    1    0
 $EndComp
@@
 L Device:R R4
 U 1 1 5FADC9DC
-P 3300 6050
-F 0 "R4" V 3093 6050 50  0000 C CNN
-F 1 "4k7" V 3184 6050 50  0000 C CNN
-F 2 "Resistor_SMD:R_0603_1608Metric_Pad0.98x0.95mm_HandSolder" V 3230 6050 50  0001 C CNN
-F 3 "~" H 3300 6050 50  0001 C CNN
-	1    3300 6050
+P 2200 6600
+F 0 "R4" V 1993 6600 50  0000 C CNN
+F 1 "4k7" V 2084 6600 50  0000 C CNN
+F 2 "Resistor_SMD:R_0603_1608Metric_Pad0.98x0.95mm_HandSolder" V 2130 6600 50  0001 C CNN
+F 3 "~" H 2200 6600 50  0001 C CNN
+	1    2200 6600
 	0    1    1    0
 $EndComp
@@
 	9300 1300 9600 1300
 Wire Wire Line
-	2400 4800 2600 4800
-Wire Wire Line
-	2400 5250 2600 5250
-Wire Wire Line
-	2400 5700 2600 5700
-Wire Wire Line
-	3150 4800 3500 4800
-Wire Wire Line
-	3150 5250 3500 5250
-Wire Wire Line
-	3500 5250 3500 4800
-Wire Wire Line
-	3150 5700 3500 5700
-Wire Wire Line
-	3500 5700 3500 5250
-Connection ~ 3500 5250
-Wire Wire Line
-	3150 6150 3500 6150
-Wire Wire Line
-	3500 6150 3500 5700
-Connection ~ 3500 5700
-Wire Wire Line
-	3700 6300 3700 6050
-Wire Wire Line
-	3700 4700 3450 4700
-Wire Wire Line
-	3450 5150 3700 5150
-Connection ~ 3700 5150
-Wire Wire Line
-	3700 5150 3700 4700
-Wire Wire Line
-	3450 5600 3700 5600
-Connection ~ 3700 5600
-Wire Wire Line
-	3700 5600 3700 5150
-Wire Wire Line
-	3450 6050 3700 6050
-Connection ~ 3700 6050
-Wire Wire Line
-	3700 6050 3700 5600
-Wire Wire Line
-	3150 4700 2600 4700
-Wire Wire Line
-	2600 4700 2600 4800
-Connection ~ 2600 4800
-Wire Wire Line
-	2600 4800 2750 4800
-Wire Wire Line
-	3150 5150 2600 5150
-Wire Wire Line
-	2600 5150 2600 5250
-Connection ~ 2600 5250
-Wire Wire Line
-	2600 5250 2750 5250
-Wire Wire Line
-	3150 5600 2600 5600
-Wire Wire Line
-	2600 5600 2600 5700
+	1300 5350 1500 5350
+Wire Wire Line
+	1300 5800 1500 5800
+Wire Wire Line
+	1300 6250 1500 6250
+Wire Wire Line
+	2050 5350 2400 5350
+Wire Wire Line
+	2050 5800 2400 5800
+Wire Wire Line
+	2400 5800 2400 5350
+Wire Wire Line
+	2050 6250 2400 6250
+Wire Wire Line
+	2400 6250 2400 5800
+Connection ~ 2400 5800
+Wire Wire Line
+	2050 6700 2400 6700
+Wire Wire Line
+	2400 6700 2400 6250
+Connection ~ 2400 6250
+Wire Wire Line
+	2600 6850 2600 6600
+Wire Wire Line
+	2600 5250 2350 5250
+Wire Wire Line
+	2350 5700 2600 5700
 Connection ~ 2600 5700
 Wire Wire Line
-	2600 5700 2750 5700
-Wire Wire Line
-	2400 6150 2600 6150
+	2600 5700 2600 5250
+Wire Wire Line
+	2350 6150 2600 6150
+Connection ~ 2600 6150
+Wire Wire Line
+	2600 6150 2600 5700
+Wire Wire Line
+	2350 6600 2600 6600
+Connection ~ 2600 6600
+Wire Wire Line
+	2600 6600 2600 6150
+Wire Wire Line
+	2050 5250 1500 5250
+Wire Wire Line
+	1500 5250 1500 5350
+Connection ~ 1500 5350
+Wire Wire Line
+	1500 5350 1650 5350
+Wire Wire Line
+	2050 5700 1500 5700
+Wire Wire Line
+	1500 5700 1500 5800
+Connection ~ 1500 5800
+Wire Wire Line
+	1500 5800 1650 5800
+Wire Wire Line
+	2050 6150 1500 6150
+Wire Wire Line
+	1500 6150 1500 6250
+Connection ~ 1500 6250
+Wire Wire Line
+	1500 6250 1650 6250
+Wire Wire Line
+	1300 6700 1500 6700
 $Comp
 L Driver_LED:TLC59108xPW U2
@@
 NoConn ~ 9100 2300
 Wire Wire Line
-	3150 6050 2600 6050
-Wire Wire Line
-	2600 6050 2600 6150
-Connection ~ 2600 6150
-Wire Wire Line
-	2600 6150 2750 6150
-Wire Wire Line
-	3500 4450 3500 4800
-Connection ~ 3500 4800
+	2050 6600 1500 6600
+Wire Wire Line
+	1500 6600 1500 6700
+Connection ~ 1500 6700
+Wire Wire Line
+	1500 6700 1650 6700
+Wire Wire Line
+	2400 5000 2400 5350
+Connection ~ 2400 5350
 Wire Wire Line
 	7350 3850 7350 3300
@@
 NoConn ~ 1300 2300
 NoConn ~ 1300 2400
+Text GLabel 1450 2600 2    39   Output ~ 0
+RST
+Wire Wire Line
+	1450 2600 1300 2600
+$Comp
+L 74xGxx:74LVC1G10 U3
+U 1 1 5FD78A6F
+P 1750 4100
+F 0 "U3" H 1750 3808 50  0000 C CNN
+F 1 "74LVC1G10" H 1750 3899 50  0000 C CNN
+F 2 "Package_TO_SOT_SMD:SOT-363_SC-70-6_Handsoldering" H 1750 4100 50  0001 C CNN
+F 3 "http://www.ti.com/lit/sg/scyt129e/scyt129e.pdf" H 1750 4100 50  0001 C CNN
+F 4 "https://www.digikey.de/product-detail/de/texas-instruments/SN74LVC1G10DCKR/296-17844-1-ND/739463" H 1750 4100 50  0001 C CNN "Digikey"
+	1    1750 4100
+	-1   0    0    1
+$EndComp
+Text GLabel 2200 4000 2    39   Input ~ 0
+Switch2
+Text GLabel 2200 4200 2    39   Input ~ 0
+Switch3
+Text GLabel 1300 4100 0    39   Input ~ 0
+RST
+Wire Wire Line
+	1450 4100 1300 4100
+Wire Wire Line
+	2200 4000 2050 4000
+Wire Wire Line
+	2200 4100 2050 4100
+Wire Wire Line
+	2200 4200 2050 4200
+Text GLabel 2200 4100 2    39   Input ~ 0
+Switch1
 $EndSCHEMATC

Commit message: Set Rext for LED current based on datasheet
Using default values, Rext for 20 mA is 600 Ohm. We're using 520 Ohm
for a safety margin.
Parts:
- R5, R6: value Rext -> 520
Changed lines of the file:
@@
 P 7700 2050
 F 0 "R5" H 7630 2004 50  0000 R CNN
-F 1 "Rext" H 7630 2095 50  0000 R CNN
+F 1 "520" H 7630 2095 50  0000 R CNN
 F 2 "Resistor_SMD:R_0603_1608Metric_Pad0.98x0.95mm_HandSolder" V 7630 2050 50  0001 C CNN
 F 3 "~" H 7700 2050 50  0001 C CNN
@@
 P 7700 4200
 F 0 "R6" H 7630 4154 50  0000 R CNN
-F 1 "Rext" H 7630 4245 50  0000 R CNN
+F 1 "520" H 7630 4245 50  0000 R CNN
 F 2 "Resistor_SMD:R_0603_1608Metric_Pad0.98x0.95mm_HandSolder" V 7630 4200 50  0001 C CNN
 F 3 "~" H 7700 4200 50  0001 C CNN

Commit message: Connect LED Driver reset to uC
Parts:
- added R7: 4k7, Resistor_SMD:R_0603_1608Metric_Pad0.98x0.95mm_HandSolder, symbol Device:R
Connections:
- net VCC: now also R7.2; no longer U1.17 (~RESET), U2.17 (~RESET)
- net LedRST: now reaches J1.12 (Pin_12)
- net LedRST: now also U1.17 (~RESET), U2.17 (~RESET), R7.1
- no-connect marks 17 -> 16
Other:
- moved on the sheet: C1, C2, R5, R6
Changed lines of the file:
@@
 L Device:C C1
 U 1 1 5FAE3E07
-P 7350 1850
-F 0 "C1" H 7465 1896 50  0000 L CNN
-F 1 "100n" H 7465 1805 50  0000 L CNN
-F 2 "Capacitor_SMD:C_0603_1608Metric_Pad1.08x0.95mm_HandSolder" H 7388 1700 50  0001 C CNN
-F 3 "~" H 7350 1850 50  0001 C CNN
-	1    7350 1850
+P 7200 1850
+F 0 "C1" H 7315 1896 50  0000 L CNN
+F 1 "100n" H 7315 1805 50  0000 L CNN
+F 2 "Capacitor_SMD:C_0603_1608Metric_Pad1.08x0.95mm_HandSolder" H 7238 1700 50  0001 C CNN
+F 3 "~" H 7200 1850 50  0001 C CNN
+	1    7200 1850
 	1    0    0    -1
 $EndComp
@@
 	8600 1100 8600 1150
 Wire Wire Line
-	8100 1600 8000 1600
-Wire Wire Line
 	8000 1150 8600 1150
-Wire Wire Line
-	8000 1150 8000 1600
 Connection ~ 8600 1150
 Wire Wire Line
@@
 L Device:R R5
 U 1 1 5FB26FE3
-P 7700 2050
-F 0 "R5" H 7630 2004 50  0000 R CNN
-F 1 "520" H 7630 2095 50  0000 R CNN
-F 2 "Resistor_SMD:R_0603_1608Metric_Pad0.98x0.95mm_HandSolder" V 7630 2050 50  0001 C CNN
-F 3 "~" H 7700 2050 50  0001 C CNN
-	1    7700 2050
+P 7550 2050
+F 0 "R5" H 7480 2004 50  0000 R CNN
+F 1 "520" H 7480 2095 50  0000 R CNN
+F 2 "Resistor_SMD:R_0603_1608Metric_Pad0.98x0.95mm_HandSolder" V 7480 2050 50  0001 C CNN
+F 3 "~" H 7550 2050 50  0001 C CNN
+	1    7550 2050
 	-1   0    0    1
 $EndComp
 Wire Wire Line
-	8100 2300 7700 2300
-Wire Wire Line
-	7700 2300 7700 2200
-Wire Wire Line
-	7700 1900 7700 1150
-Wire Wire Line
-	7700 1150 8000 1150
-Connection ~ 8000 1150
+	8100 2300 7550 2300
+Wire Wire Line
+	7550 2300 7550 2200
+Wire Wire Line
+	7550 1900 7550 1150
+Wire Wire Line
+	7550 1150 8000 1150
 Text GLabel 7900 1700 0    39   BiDi ~ 0
 SCL
@@
 Wire Wire Line
 	8100 1900 8000 1900
-Wire Wire Line
-	8000 1900 8000 1600
-Connection ~ 8000 1600
 $Comp
 L Device:LED_ARGB D1
@@
 L Device:C C2
 U 1 1 5FBB8133
-P 7350 4000
-F 0 "C2" H 7465 4046 50  0000 L CNN
-F 1 "100n" H 7465 3955 50  0000 L CNN
-F 2 "Capacitor_SMD:C_0603_1608Metric_Pad1.08x0.95mm_HandSolder" H 7388 3850 50  0001 C CNN
-F 3 "~" H 7350 4000 50  0001 C CNN
-	1    7350 4000
+P 7200 4000
+F 0 "C2" H 7315 4046 50  0000 L CNN
+F 1 "100n" H 7315 3955 50  0000 L CNN
+F 2 "Capacitor_SMD:C_0603_1608Metric_Pad1.08x0.95mm_HandSolder" H 7238 3850 50  0001 C CNN
+F 3 "~" H 7200 4000 50  0001 C CNN
+	1    7200 4000
 	1    0    0    -1
 $EndComp
@@
 	8600 4650 8600 4700
 Wire Wire Line
-	8100 3750 8000 3750
-Wire Wire Line
 	8000 3300 8600 3300
-Wire Wire Line
-	8000 3300 8000 3750
 Connection ~ 8600 3300
 Wire Wire Line
@@
 	8100 4350 8000 4350
 Connection ~ 8000 4350
-Wire Wire Line
-	8000 4350 8000 4700
 $Comp
 L Device:R R6
 U 1 1 5FBB8151
-P 7700 4200
-F 0 "R6" H 7630 4154 50  0000 R CNN
-F 1 "520" H 7630 4245 50  0000 R CNN
-F 2 "Resistor_SMD:R_0603_1608Metric_Pad0.98x0.95mm_HandSolder" V 7630 4200 50  0001 C CNN
-F 3 "~" H 7700 4200 50  0001 C CNN
-	1    7700 4200
+P 7550 4200
+F 0 "R6" H 7480 4154 50  0000 R CNN
+F 1 "520" H 7480 4245 50  0000 R CNN
+F 2 "Resistor_SMD:R_0603_1608Metric_Pad0.98x0.95mm_HandSolder" V 7480 4200 50  0001 C CNN
+F 3 "~" H 7550 4200 50  0001 C CNN
+	1    7550 4200
 	-1   0    0    1
 $EndComp
 Wire Wire Line
-	8100 4450 7700 4450
-Wire Wire Line
-	7700 4450 7700 4350
-Wire Wire Line
-	7700 4050 7700 3300
-Wire Wire Line
-	7700 3300 8000 3300
-Connection ~ 8000 3300
+	8100 4450 7550 4450
+Wire Wire Line
+	7550 4450 7550 4350
+Wire Wire Line
+	7550 4050 7550 3300
+Wire Wire Line
+	7550 3300 8000 3300
 Text GLabel 7900 3850 0    39   BiDi ~ 0
 SCL
@@
 Wire Wire Line
 	8100 4050 8000 4050
-Wire Wire Line
-	8000 4050 8000 3750
-Connection ~ 8000 3750
 $Comp
 L Device:LED_ARGB D4
@@
 Connection ~ 2400 5350
 Wire Wire Line
-	7350 3850 7350 3300
-Wire Wire Line
-	7350 3300 7700 3300
-Connection ~ 7700 3300
-Wire Wire Line
-	7350 4150 7350 4700
-Wire Wire Line
-	7350 4700 8000 4700
-Connection ~ 8000 4700
-Wire Wire Line
-	7350 1700 7350 1150
-Wire Wire Line
-	7350 1150 7700 1150
-Connection ~ 7700 1150
-Wire Wire Line
-	7350 2000 7350 2550
-Wire Wire Line
-	7350 2550 8000 2550
-Connection ~ 8000 2550
+	7200 3850 7200 3300
+Wire Wire Line
+	7200 3300 7550 3300
+Connection ~ 7550 3300
+Wire Wire Line
+	7200 4150 7200 4700
+Wire Wire Line
+	7200 4700 8000 4700
+Wire Wire Line
+	7200 1700 7200 1150
+Wire Wire Line
+	7200 1150 7550 1150
+Connection ~ 7550 1150
+Wire Wire Line
+	7200 2000 7200 2550
+Wire Wire Line
+	7200 2550 8000 2550
 Wire Wire Line
 	8600 2550 8600 2650
@@
 NoConn ~ 2500 1900
 NoConn ~ 2500 1800
-NoConn ~ 2500 1700
 Wire Wire Line
 	3750 1750 3750 1850
@@
 Text GLabel 2200 4100 2    39   Input ~ 0
 Switch1
+Connection ~ 8000 2550
+Connection ~ 8000 1150
+Wire Wire Line
+	8000 4350 8000 4700
+Connection ~ 8000 4700
+Connection ~ 8000 3300
+Text GLabel 7900 1600 0    39   Input ~ 0
+LedRST
+Wire Wire Line
+	8000 1150 8000 1900
+Wire Wire Line
+	7900 1600 8100 1600
+Text GLabel 7900 3750 0    39   Input ~ 0
+LedRST
+Wire Wire Line
+	8000 3300 8000 4050
+Wire Wire Line
+	7900 3750 8100 3750
+Text GLabel 2800 1700 2    39   Output ~ 0
+LedRST
+Wire Wire Line
+	2500 1700 2700 1700
+$Comp
+L Device:R R7
+U 1 1 5FB9F7A1
+P 2700 1550
+F 0 "R7" H 2630 1504 50  0000 R CNN
+F 1 "4k7" H 2630 1595 50  0000 R CNN
+F 2 "Resistor_SMD:R_0603_1608Metric_Pad0.98x0.95mm_HandSolder" V 2630 1550 50  0001 C CNN
+F 3 "~" H 2700 1550 50  0001 C CNN
+	1    2700 1550
+	-1   0    0    1
+$EndComp
+Connection ~ 2700 1700
+Wire Wire Line
+	2700 1700 2800 1700
+$Comp
+L power:VCC #PWR03
+U 1 1 5FBA1249
+P 2700 1350
+F 0 "#PWR03" H 2700 1200 50  0001 C CNN
+F 1 "VCC" H 2715 1523 50  0000 C CNN
+F 2 "" H 2700 1350 50  0001 C CNN
+F 3 "" H 2700 1350 50  0001 C CNN
+	1    2700 1350
+	1    0    0    -1
+$EndComp
+Wire Wire Line
+	2700 1350 2700 1400
 $EndSCHEMATC
